File: pika_go_0/audio.kicad_sch (KiCad schematic)
At the start: 22 parts, among them J7 MIC, J8 SPK, U4 SSM2305RMZ-REEL7, U5 MAX4467EKA_T

Commit message: Libraries cleanup, schematics finished, copper tracing finished, still need some PCB cleanup
Parts:
- U4: symbol ton_library:SSM2305RMZ-REEL7 -> Pika:SSM2305RMZ-REEL7
- U5: symbol ton_library:MAX4467EKA_T -> Pika:MAX4467EKA_T

Commit message: Some capacitors footprints changed, minor cleanup
Parts:
- C31: footprint Capacitor_SMD:C_0805_2012Metric_Pad1.18x1.45mm_HandSolder -> Capacitor_SMD:C_0603_1608Metric_Pad1.08x0.95mm_HandSolder; MP (none) -> GRM188Z71A106KA73D
Changed lines of the file:
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@@
 			)
 		)
-		(property "Footprint" "Capacitor_SMD:C_0805_2012Metric_Pad1.18x1.45mm_HandSolder"
+		(property "Footprint" "Capacitor_SMD:C_0603_1608Metric_Pad1.08x0.95mm_HandSolder"
 			(at 152.0952 41.91 0)
 			(hide yes)
@@
 			(at 151.13 38.1 0)
 			(hide yes)
+			(show_name no)
+			(do_not_autoplace no)
+			(effects
+				(font
+					(size 1.27 1.27)
+				)
+			)
+		)
+		(property "MP" "GRM188Z71A106KA73D"
+			(at 151.13 38.1 0)
+			(hide yes)

Commit message: Schematic reannotated, cleanup
Parts:
- C39: renamed from C22; MP (none) -> CL10C470JB8NNNC
- C40: renamed from C23; MP (none) -> C0603C104K5RACTU
- C41: renamed from C24; MP (none) -> CL10A105KB8NNNC
- C42: renamed from C25; MP (none) -> C0603C104K5RACTU
- C43: renamed from C26; MP (none) -> C0603C104K5RACTU
- C44: renamed from C27; MP (none) -> C0603C104K5RACTU
- C45: renamed from C28; MP (none) -> CL10C470JB8NNNC
- C46: renamed from C29; MP (none) -> C0603C104K5RACTU
- C47: renamed from C30; MP (none) -> C0603C104K5RACTU
- J7, J8: MP (none) -> 0532610271
- R21: renamed from R14; MP (none) -> RC0603FR-072K2L
- R22: renamed from R15; MP (none) -> RC0603FR-0720KL
- R23: renamed from R16; MP (none) -> RC0603FR-071KL
- R24: renamed from R17; MP (none) -> RC0603FR-07100KL
- R25: renamed from R18; MP (none) -> RC0603FR-07100KL
- R26: renamed from R19; MP (none) -> RC0603FR-07100KL
- R27: renamed from R20; MP (none) -> RC0603FR-07100KL
- R28: renamed from R21; MP (none) -> RC0603FR-07200KL
- U9: renamed from U4; MP (none) -> SSM2305RMZ-REEL7
- renumbered C31 to C48, U5 to U10
