File: pika_go_0/gnss.kicad_sch (KiCad schematic)
At the start: 2 parts, among them U7 CAM-M8Q-0

Commit message: Libraries cleanup, schematics finished, copper tracing finished, still need some PCB cleanup
Parts:
- U7: footprint ton_library:LCC100P960X1400X210-31N -> Pika:LCC100P960X1400X210-31N; symbol ton_library:CAM-M8Q-0 -> Pika:CAM-M8Q-0
Changed lines of the file:
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@@
+			)
+		)
+		(property "MANUFACTURER_PART_NUMBER" ""
+			(at 99.06 30.48 0)
+			(hide yes)
+			(show_name no)
+			(do_not_autoplace no)
+			(effects
+				(font
+					(size 1.27 1.27)
+				)
+			)
+		)
+		(property "MFR_NAME" ""
+			(at 99.06 30.48 0)
+			(hide yes)
+			(show_name no)
+			(do_not_autoplace no)
+			(effects
+				(font
+					(size 1.27 1.27)
+				)
 			)
 		)
@@
 	)
 	(symbol
-		(lib_id "ton_library:CAM-M8Q-0")
+		(lib_id "Pika:CAM-M8Q-0")
 		(at 58.42 41.91 0)
 		(unit 1)
@@
 			)
 		)
-		(property "Footprint" "ton_library:LCC100P960X1400X210-31N"
+		(property "Footprint" "Pika:LCC100P960X1400X210-31N"
 			(at 58.42 41.91 0)
 			(hide yes)
@@
 			)
 		)
+		(property "MANUFACTURER_PART_NUMBER" ""
+			(at 58.42 41.91 0)
+			(hide yes)
+			(show_name no)
+			(do_not_autoplace no)
+			(effects
+				(font
+					(size 1.27 1.27)
+				)
+			)
+		)
+		(property "MFR_NAME" ""
+			(at 58.42 41.91 0)
+			(hide yes)
+			(show_name no)
+			(do_not_autoplace no)
+			(effects
+				(font
+					(size 1.27 1.27)
+				)
+			)
+		)

Commit message: Schematic reannotated, cleanup
Parts:
- C38: renamed from C34; MP (none) -> C0603C104K5RACTU
- renumbered U7 to U8
Changed lines of the file:
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@@
 		(dnp no)
 		(fields_autoplaced yes)
-		(property "Reference" "#PWR078"
+		(property "Reference" "#PWR091"
 			(at 99.06 40.64 0)
 			(hide yes)
@@
 			(project "pika_go_0"
 				(path "/71487f0a-8ca7-4aa8-8af1-384680074486/b714831d-7c84-4e82-80fc-c753a31ecf3a"
-					(reference "#PWR078")
+					(reference "#PWR091")
 					(unit 1)
 				)
@@
 		(dnp no)
 		(fields_autoplaced yes)
-		(property "Reference" "#PWR077"
+		(property "Reference" "#PWR090"
 			(at 86.36 63.5 0)
 			(hide yes)
@@
 			(project "pika_go_0"
 				(path "/71487f0a-8ca7-4aa8-8af1-384680074486/b714831d-7c84-4e82-80fc-c753a31ecf3a"
-					(reference "#PWR077")
+					(reference "#PWR090")
 					(unit 1)
 				)
@@
 		(in_pos_files yes)
 		(dnp no)
-		(property "Reference" "#PWR079"
+		(property "Reference" "#PWR092"
 			(at 101.6 26.67 0)
 			(hide yes)
@@
 			(project "pika_go_0"
 				(path "/71487f0a-8ca7-4aa8-8af1-384680074486/b714831d-7c84-4e82-80fc-c753a31ecf3a"
-					(reference "#PWR079")
+					(reference "#PWR092")
 					(unit 1)
 				)
@@
 		(dnp no)
 		(fields_autoplaced yes)
-		(property "Reference" "C34"
+		(property "Reference" "C38"
 			(at 102.87 29.2099 0)
 			(show_name no)
@@
 		)
 		(property "MFR_NAME" ""
+			(at 99.06 30.48 0)
+			(hide yes)
+			(show_name no)
+			(do_not_autoplace no)
+			(effects
+				(font
+					(size 1.27 1.27)
+				)
+			)
+		)
+		(property "MP" "C0603C104K5RACTU"
 			(at 99.06 30.48 0)
 			(hide yes)
@@
 			(project "pika_go_0"
 				(path "/71487f0a-8ca7-4aa8-8af1-384680074486/b714831d-7c84-4e82-80fc-c753a31ecf3a"
-					(reference "C34")
+					(reference "C38")
 					(unit 1)
 				)
@@
 		(dnp no)
 		(fields_autoplaced yes)
-		(property "Reference" "U7"
+		(property "Reference" "U8"
 			(at 58.42 19.05 0)
 			(show_name no)
@@
 			(project "pika_go_0"
 				(path "/71487f0a-8ca7-4aa8-8af1-384680074486/b714831d-7c84-4e82-80fc-c753a31ecf3a"
-					(reference "U7")
+					(reference "U8")
 					(unit 1)
 				)
