File: pika_go_0/power.kicad_sch (KiCad schematic)
At the start: 31 parts, among them J2 BAT, U11 TPS610333DRLR, U13 BQ25895RTW, U9 MCP1703Ax-330xxMB

Commit message: Some capacitors footprints changed, minor cleanup
Parts:
- C3, C4, C61, C70, C71: footprint Capacitor_SMD:C_1210_3225Metric_Pad1.33x2.70mm_HandSolder -> Capacitor_SMD:C_0805_2012Metric_Pad1.18x1.45mm_HandSolder; MP (none) -> CL21A226KOQNNNG
- C6, C9: footprint Capacitor_SMD:C_1210_3225Metric_Pad1.33x2.70mm_HandSolder -> Capacitor_SMD:C_0603_1608Metric_Pad1.08x0.95mm_HandSolder; MP (none) -> GRM188Z71A106KA73D
- L3: value 2.2u -> 1u; footprint Inductor_SMD:L_1210_3225Metric_Pad1.42x2.65mm_HandSolder -> Pika:L_ABRACON_AMELH4018S; MP (none) -> AMELH4018S-1R0MT
- R2: value 260 -> 261
Changed lines of the file:
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@@
 			)
 		)
-		(property "Footprint" "Capacitor_SMD:C_1210_3225Metric_Pad1.33x2.70mm_HandSolder"
+		(property "Footprint" "Capacitor_SMD:C_0805_2012Metric_Pad1.18x1.45mm_HandSolder"
 			(at 119.0752 63.5 0)
 			(hide yes)
@@
 			)
 		)
+		(property "MP" "CL21A226KOQNNNG"
+			(at 118.11 67.31 0)
+			(hide yes)
+			(show_name no)
+			(do_not_autoplace no)
+			(effects
+				(font
+					(size 1.27 1.27)
+				)
+			)
+		)
 		(pin "1"
 		)
@@
 			)
 		)
-		(property "Value" "2.2u"
+		(property "Value" "1u"
 			(at 109.22 58.4199 0)
 			(show_name no)
@@
 			)
 		)
-		(property "Footprint" "Inductor_SMD:L_1210_3225Metric_Pad1.42x2.65mm_HandSolder"
+		(property "Footprint" "Pika:L_ABRACON_AMELH4018S"
 			(at 106.68 57.15 0)
 			(hide yes)
@@
 			)
 		)
-		(property "MP" ""
-			(at 106.68 57.15 0)
-			(hide yes)
-			(show_name no)
-			(do_not_autoplace no)
-			(effects
-				(font
-					(size 1.27 1.27)
-				)
-			)
-		)
-		(property "MANUFACTURER_PART_NUMBER" ""
-			(at 106.68 57.15 0)
-			(hide yes)
-			(show_name no)
-			(do_not_autoplace no)
-			(effects
-				(font
-					(size 1.27 1.27)
-				)
-			)
-		)
-		(property "MFR_NAME" ""
+		(property "MP" "AMELH4018S-1R0MT"
 			(at 106.68 57.15 0)
 			(hide yes)
@@
 			)
 		)
-		(property "Footprint" "Capacitor_SMD:C_1210_3225Metric_Pad1.33x2.70mm_HandSolder"
+		(property "Footprint" "Capacitor_SMD:C_0805_2012Metric_Pad1.18x1.45mm_HandSolder"
 			(at 133.0452 133.35 0)
 			(hide yes)
@@
 			)
 		)
+		(property "MP" "CL21A226KOQNNNG"
+			(at 132.08 137.16 0)
+			(hide yes)
+			(show_name no)
+			(do_not_autoplace no)
+			(effects
+				(font
+					(size 1.27 1.27)
+				)
+			)
+		)
 		(pin "1"
 		)
@@
 			)
 		)
-		(property "Footprint" "Capacitor_SMD:C_1210_3225Metric_Pad1.33x2.70mm_HandSolder"
+		(property "Footprint" "Capacitor_SMD:C_0805_2012Metric_Pad1.18x1.45mm_HandSolder"
 			(at 42.2148 135.89 0)
 			(hide yes)
@@
 			)
 		)
+		(property "MP" "CL21A226KOQNNNG"
+			(at 43.18 132.08 0)
+			(hide yes)
+			(show_name no)
+			(do_not_autoplace no)
+			(effects
+				(font
+					(size 1.27 1.27)
+				)
+			)
+		)
 		(pin "1"
 		)
@@
 			)
 		)
-		(property "Footprint" "Capacitor_SMD:C_1210_3225Metric_Pad1.33x2.70mm_HandSolder"
+		(property "Footprint" "Capacitor_SMD:C_0805_2012Metric_Pad1.18x1.45mm_HandSolder"
 			(at 107.6452 63.5 0)
 			(hide yes)
@@
 			)
 		)
+		(property "MP" "CL21A226KOQNNNG"
+			(at 106.68 67.31 0)
+			(hide yes)
+			(show_name no)
+			(do_not_autoplace no)
+			(effects
+				(font
+					(size 1.27 1.27)
+				)
+			)
+		)
 		(pin "1"
 		)
@@
 			)
 		)
-		(property "Value" "260"
+		(property "Value" "261"
 			(at 64.77 80.01 90)
 			(show_name no)
@@
 			)
 		)
-		(property "Footprint" "Capacitor_SMD:C_1210_3225Metric_Pad1.33x2.70mm_HandSolder"
+		(property "Footprint" "Capacitor_SMD:C_0805_2012Metric_Pad1.18x1.45mm_HandSolder"
 			(at 121.6152 133.35 0)
 			(hide yes)
@@
 			)
 		)
+		(property "MP" "CL21A226KOQNNNG"
+			(at 120.65 137.16 0)
+			(hide yes)
+			(show_name no)
+			(do_not_autoplace no)
+			(effects
+				(font
+					(size 1.27 1.27)
+				)
+			)
+		)
 		(pin "1"
 		)
@@
 			)
 		)
-		(property "Footprint" "Capacitor_SMD:C_1210_3225Metric_Pad1.33x2.70mm_HandSolder"
+		(property "Footprint" "Capacitor_SMD:C_0603_1608Metric_Pad1.08x0.95mm_HandSolder"
 			(at 119.0752 48.26 0)
 			(hide yes)
@@
 			)
 		)
+		(property "MP" "GRM188Z71A106KA73D"
+			(at 118.11 52.07 0)
+			(hide yes)
+			(show_name no)
+			(do_not_autoplace no)
+			(effects
+				(font
+					(size 1.27 1.27)
+				)
+			)
+		)
 		(pin "1"
 		)
@@
 			)
 		)
-		(property "Footprint" "Capacitor_SMD:C_1210_3225Metric_Pad1.33x2.70mm_HandSolder"
+		(property "Footprint" "Capacitor_SMD:C_0603_1608Metric_Pad1.08x0.95mm_HandSolder"
 			(at 148.8948 48.26 0)
 			(hide yes)
@@
 			(at 149.86 44.45 0)
 			(hide yes)
+			(show_name no)
+			(do_not_autoplace no)
+			(effects
+				(font
+					(size 1.27 1.27)
+				)
+			)
+		)
+		(property "MP" "GRM188Z71A106KA73D"
+			(at 149.86 44.45 0)
+			(hide yes)

Commit message: Schematic reannotated, cleanup
Parts:
- C10: renamed from C72; MP (none) -> C0603C104K5RACTU
- C11: renamed from C7; MP (none) -> CL10A475KO8NNNC
- C13: renamed from C69; MP (none) -> CL10A475KO8NNNC
- C2: renamed from C64; MP (none) -> C0603C104K5RACTU
- C3: renamed from C5; MP (none) -> CL10A105KB8NNNC
- C4: renamed from C36; MP (none) -> CL10B473KB8NNNC
- D1: MP (none) -> LTST-C190KGKT
- FB1: renamed from FB4; MP (none) -> 2508056017Y2
- J1: renamed from J2; MP (none) -> S3B-PH-K-S
- R1: renamed from R5; MP (none) -> RC0603FR-0710KL
- R2: renamed from R6; MP (none) -> RC0603FR-0710KL
- R3: renamed from R9; MP (none) -> RC0603FR-0710KL
- R4: renamed from R2; MP (none) -> RC0603FR-07261RL
- R5: renamed from R31; now left out of the parts list
- R6: renamed from R27; MP (none) -> RC0603FR-0710KL
- R7: renamed from R1; MP (none) -> ERJ-3EKF3301V
- R8: renamed from R3; MP (none) -> RC0603FR-075K23L; Tolerance (none) -> 1%
- R9: renamed from R4; MP (none) -> RC0603FR-0730K1L; Tolerance (none) -> 1%
- U1: renamed from U11; MP (none) -> TPS610333DRLR
- U2: renamed from U13; MP (none) -> BQ25895RTWT
- U3: renamed from U9; MP (none) -> MCP1703AT-3302E/MB
- renumbered C61 to C1, C9 to C12, C3 to C5, C4 to C7, C70 to C8, C71 to C9, L6 to L1, L3 to L2
