File: pika_go_0/radio.kicad_sch (KiCad schematic)
At the start: 4 parts, among them J9 ANT, U6 E22-900M30S

Commit message: Libraries cleanup, schematics finished, copper tracing finished, still need some PCB cleanup
Parts:
- U6: footprint ton_library:XCVR_E22-900M30S -> Pika:XCVR_E22-900M30S; symbol ton_library:E22-900M30S -> Pika:E22-900M30S
Changed lines of the file:
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@@
+			)
+		)
+		(property "MANUFACTURER_PART_NUMBER" ""
+			(at 132.08 31.75 0)
+			(hide yes)
+			(show_name no)
+			(do_not_autoplace no)
+			(effects
+				(font
+					(size 1.27 1.27)
+				)
+			)
+		)
+		(property "MFR_NAME" ""
+			(at 132.08 31.75 0)
+			(hide yes)
+			(show_name no)
+			(do_not_autoplace no)
+			(effects
+				(font
+					(size 1.27 1.27)
+				)
 			)
 		)
@@
 	)
 	(symbol
-		(lib_id "ton_library:E22-900M30S")
+		(lib_id "Pika:E22-900M30S")
 		(at 63.5 40.64 0)
 		(unit 1)
@@
 			)
 		)
-		(property "Footprint" "ton_library:XCVR_E22-900M30S"
+		(property "Footprint" "Pika:XCVR_E22-900M30S"
 			(at 63.5 40.64 0)
 			(hide yes)
@@
 				)
 				(justify bottom)
+			)
+		)
+		(property "MANUFACTURER_PART_NUMBER" ""
+			(at 63.5 40.64 0)
+			(hide yes)
+			(show_name no)
+			(do_not_autoplace no)
+			(effects
+				(font
+					(size 1.27 1.27)
+				)
+			)
+		)
+		(property "MFR_NAME" ""
+			(at 63.5 40.64 0)
+			(hide yes)
+			(show_name no)
+			(do_not_autoplace no)
+			(effects
+				(font
+					(size 1.27 1.27)
+				)
 			)
 		)
@@
 			)
 		)
+		(property "MANUFACTURER_PART_NUMBER" ""
+			(at 119.38 31.75 0)
+			(hide yes)
+			(show_name no)
+			(do_not_autoplace no)
+			(effects
+				(font
+					(size 1.27 1.27)
+				)
+			)
+		)
+		(property "MFR_NAME" ""
+			(at 119.38 31.75 0)
+			(hide yes)
+			(show_name no)
+			(do_not_autoplace no)
+			(effects
+				(font
+					(size 1.27 1.27)
+				)
+			)
+		)
 		(pin "2"
 		)
@@
 			(at 105.41 33.02 0)
 			(hide yes)
+			(show_name no)
+			(do_not_autoplace no)
+			(effects
+				(font
+					(size 1.27 1.27)
+				)
+			)
+		)
+		(property "MANUFACTURER_PART_NUMBER" ""
+			(at 105.41 33.02 0)
+			(hide yes)
+			(show_name no)
+			(do_not_autoplace no)
+			(effects
+				(font
+					(size 1.27 1.27)
+				)
+			)
+		)
+		(property "MFR_NAME" ""
+			(at 105.41 33.02 0)
+			(hide yes)

Commit message: More 3D models added to library. Use external SMA-U.FL cable instead in SMA connector on PCB edge.
Parts:
- removed J9: ANT, Connector_Coaxial:SMA_Molex_73251-2120_EdgeMount_Horizontal, symbol Connector:Conn_Coaxial
Connections:
- net ANT: no longer names the net of U6.21 (ANT)
- no-connect marks 0 -> 1
Other:
- note added: "RF cable: Würth Elektronik 636208040050"

Commit message: Schematic reannotated, cleanup
Parts:
- C36: renamed from C32; MP (none) -> C0603C104K5RACTU
- C37: renamed from C33; MP (none) -> CL10A475KO8NNNC
- renumbered U6 to U7
Changed lines of the file:
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@@
 		(dnp no)
 		(fields_autoplaced yes)
-		(property "Reference" "C33"
+		(property "Reference" "C37"
 			(at 135.89 30.4799 0)
 			(show_name no)
@@
 		)
 		(property "MFR_NAME" ""
+			(at 132.08 31.75 0)
+			(hide yes)
+			(show_name no)
+			(do_not_autoplace no)
+			(effects
+				(font
+					(size 1.27 1.27)
+				)
+			)
+		)
+		(property "MP" "CL10A475KO8NNNC"
 			(at 132.08 31.75 0)
 			(hide yes)
@@
 			(project "pika_go_0"
 				(path "/71487f0a-8ca7-4aa8-8af1-384680074486/5a302e3d-d282-41fb-b48e-1fbf9b3c621c"
-					(reference "C33")
+					(reference "C37")
 					(unit 1)
 				)
@@
 		(dnp no)
 		(fields_autoplaced yes)
-		(property "Reference" "U6"
+		(property "Reference" "U7"
 			(at 63.5 20.32 0)
 			(show_name no)
@@
 			(project "pika_go_0"
 				(path "/71487f0a-8ca7-4aa8-8af1-384680074486/5a302e3d-d282-41fb-b48e-1fbf9b3c621c"
-					(reference "U6")
+					(reference "U7")
 					(unit 1)
 				)
@@
 		(dnp no)
 		(fields_autoplaced yes)
-		(property "Reference" "#PWR075"
+		(property "Reference" "#PWR088"
 			(at 132.08 41.91 0)
 			(hide yes)
@@
 			(project "pika_go_0"
 				(path "/71487f0a-8ca7-4aa8-8af1-384680074486/5a302e3d-d282-41fb-b48e-1fbf9b3c621c"
-					(reference "#PWR075")
+					(reference "#PWR088")
 					(unit 1)
 				)
@@
 		(dnp no)
 		(fields_autoplaced yes)
-		(property "Reference" "#PWR076"
+		(property "Reference" "#PWR089"
 			(at 132.08 27.94 0)
 			(hide yes)
@@
 			(project "pika_go_0"
 				(path "/71487f0a-8ca7-4aa8-8af1-384680074486/5a302e3d-d282-41fb-b48e-1fbf9b3c621c"
-					(reference "#PWR076")
+					(reference "#PWR089")
 					(unit 1)
 				)
@@
 		(dnp no)
 		(fields_autoplaced yes)
-		(property "Reference" "#PWR074"
+		(property "Reference" "#PWR087"
 			(at 119.38 41.91 0)
 			(hide yes)
@@
 			(project "pika_go_0"
 				(path "/71487f0a-8ca7-4aa8-8af1-384680074486/5a302e3d-d282-41fb-b48e-1fbf9b3c621c"
-					(reference "#PWR074")
+					(reference "#PWR087")
 					(unit 1)
 				)
@@
 		(in_pos_files yes)
 		(dnp no)
-		(property "Reference" "C32"
+		(property "Reference" "C36"
 			(at 123.19 30.4799 0)
 			(show_name no)
@@
 		)
 		(property "MFR_NAME" ""
+			(at 119.38 31.75 0)
+			(hide yes)
+			(show_name no)
+			(do_not_autoplace no)
+			(effects
+				(font
+					(size 1.27 1.27)
+				)
+			)
+		)
+		(property "MP" "C0603C104K5RACTU"
 			(at 119.38 31.75 0)
 			(hide yes)
@@
 			(project "pika_go_0"
 				(path "/71487f0a-8ca7-4aa8-8af1-384680074486/5a302e3d-d282-41fb-b48e-1fbf9b3c621c"
-					(reference "C32")
+					(reference "C36")
 					(unit 1)
 				)
@@
 		(dnp no)
 		(fields_autoplaced yes)
-		(property "Reference" "#PWR072"
+		(property "Reference" "#PWR086"
 			(at 81.28 59.69 0)
 			(hide yes)
@@
 			(project "pika_go_0"
 				(path "/71487f0a-8ca7-4aa8-8af1-384680074486/5a302e3d-d282-41fb-b48e-1fbf9b3c621c"
-					(reference "#PWR072")
+					(reference "#PWR086")
 					(unit 1)
 				)
