File: pika_go_0/usb.kicad_sch (KiCad schematic)
At the start: 17 parts, among them J1 USB_C_Receptacle_USB2.0_16P, U1 MCP1703Ax-500xxTT, U8 USB3300-EZK

Commit message: Schematic reannotated, cleanup
Parts:
- C27: renamed from C41; MP (none) -> C0603C104K5RACTU
- C28: renamed from C42; MP (none) -> C0603C104K5RACTU
- C29: renamed from C44; MP (none) -> C0603C104K5RACTU
- C30: renamed from C43; MP (none) -> C0603C104K5RACTU
- C31: renamed from C37; MP (none) -> C0603C104K5RACTU
- C32: renamed from C38; MP (none) -> CL10A475KO8NNNC
- C33: renamed from C45; MP (none) -> CL10A105KB8NNNC
- C34: renamed from C39; MP (none) -> C0603C104K5RACTU
- C35: renamed from C40; MP (none) -> CL10A475KO8NNNC
- FB2: MP (none) -> 2508056017Y2
- J6: renamed from J1; MP (none) -> 12402484E512A
- R17: renamed from R8; MP (none) -> RC0603FR-07820RL; Tolerance (none) -> 1%
- R18: renamed from R7; MP (none) -> RC0603FR-0712KL
- R19: renamed from R23; MP (none) -> RMCF0603FT5K10
- R20: renamed from R24; MP (none) -> RMCF0603FT5K10
- U5: renamed from U8; MP (none) -> USB3300-EZK
- U6: renamed from U1; MP (none) -> MCP1703AT-5002E/CB
