File: pika_go_0/mcu.kicad_sch (KiCad schematic)
At the start: 34 parts, among them J3 MCU_DEBUG, J4 SD_CARD, J5 Conn_01x02, J6 LCD, Q1 BSS138, SW1 LSN, SW2 PTT, SW3 UP, SW4 DOWN, SW5 LEFT, SW6 RIGHT, SW7 PWR, U3 STM32H733VGTx, Y1 SG-210STF 24.0000ML0

Commit message: Libraries cleanup, schematics finished, copper tracing finished, still need some PCB cleanup
Parts:
- removed C21: 100n, Capacitor_SMD:C_0603_1608Metric_Pad1.08x0.95mm_HandSolder, symbol Device:C
- removed J4: SD_CARD, ton_library:503182-1852_MOL, symbol ton_library:5031821852
- added C46: 100n, Capacitor_SMD:C_0603_1608Metric_Pad1.08x0.95mm_HandSolder, symbol Device:C
- added D2: BAT54WS, Diode_SMD:D_SOD-323_HandSoldering, symbol Diode:BAT54J
- added J4: Micro_SD_Card_Det1, Pika:CUI_MSD-1-A, symbol Connector:Micro_SD_Card_Det1
- J6: footprint ton_library:527461471_MOL -> Pika:527461471_MOL
- SW3, SW4, SW5, SW6: footprint ton_library:TE_STSA -> Pika:TE_STSA
Connections:
- net +3.3V: now also C46.1, J4.4 (VDD)
- net BTN_PWR: now also D2.1 (K); no longer U3.40 (PE10)
- net GND: now also C46.2, J4.6 (VSS), J4.SH (SHIELD)
- net SD_CK: now also J4.5 (CLK)
- net SD_CMD: now also J4.3 (CMD)
- net SD_D0: now also J4.7 (DAT0)
- net SD_D1: now also J4.8 (DAT1)
- net SD_D2: now also J4.1 (DAT2)
- net SD_D3: now also J4.2 (DAT3/CD)
- net CHG_CD: no longer names the net of U3.96 (PB9)
- net CHG_PSEL: no longer names the net of U3.95 (PB8)
- new net: D2.2 (A), U3.40 (PE10)
Other:
- note added: "When MCU is not powered it may pull QON pin of the battery charger IC down, diode prevents this."
- moved on the sheet: J3

Commit message: Schematic reannotated, cleanup
Parts:
- C14: renamed from C10; MP (none) -> C0603C104K5RACTU
- C15: renamed from C35; MP (none) -> C0603C104K5RACTU
- C16: renamed from C11; MP (none) -> C0603C104K5RACTU
- C17: renamed from C12; MP (none) -> C0603C104K5RACTU
- C18: renamed from C13; MP (none) -> C0603C104K5RACTU
- C19: renamed from C14; MP (none) -> C0603C104K5RACTU
- C20: renamed from C15; MP (none) -> CL10A225KP8NNNC
- C21: renamed from C16; MP (none) -> C0603C104K5RACTU
- C22: renamed from C17; MP (none) -> C0603C104K5RACTU
- C23: renamed from C18; MP (none) -> CL10A475KO8NNNC
- C24: renamed from C19; MP (none) -> C0603C104K5RACTU
- C25: renamed from C20; MP (none) -> CL10A475KO8NNNC
- C26: renamed from C46; MP (none) -> C0603C104K5RACTU
- D2: MP (none) -> BAT54WS-7-F
- J2: renamed from J3; MP (none) -> SM06B-SRSS-TB
- J4: renamed from J5; MP (none) -> SM02B-SRSS-TB
- J5: renamed from J6; MP (none) -> 0527461471
- Q1: MP (none) -> BSS138
- R10: renamed from R22; MP (none) -> RC0603FR-0710KL
- R11: renamed from R26; MP (none) -> ERJ-3EKF22R0V
- R12: renamed from R25; MP (none) -> ERJ-3EKF22R0V
- R13: renamed from R10; MP (none) -> RC0603FR-0710KL
- R14: renamed from R12; MP (none) -> RC0603FR-0710KL
- R15: renamed from R11; MP (none) -> RC0603FR-0710KL
- R16: renamed from R13; MP (none) -> RC0603FR-0710KL
- U4: renamed from U3; MP (none) -> STM32H733VGT6
- renumbered J4 to J3, SW7 to SW1, SW1 to SW2, SW2 to SW3, SW3 to SW4, SW4 to SW5, SW5 to SW6, SW6 to SW7

Commit message: Silk screen cleanup, various fixes after DRC
Parts:
- J4: value Conn_01x02 -> BKLT
